File: pcb/lmcl_board/lmcl_board.sch (EAGLE design)
At the start: 57 parts, among them CN1 B2B-PH-K-S, IC1 V7805-1000, K1 61400416021, U1 SFW15R-1STE1LF, U2 SFW15R-1STE1LF, U3 DMG1012T, U4 TENDA_P200, U5 PAM2306AYPKE, U6 AP7115-25SEG

Commit message: lmcl_board
Parts:
- removed C10: 4.7u, resistor:C-EUC0603
- removed C11: 22u, resistor:CPOL-EU153CLV-0405
- removed C12, C13, C14: 47u, resistor:C-EUC1206
- removed C15: 10u, resistor:CPOL-EU153CLV-0405
- removed C16, C8: 1u, resistor:C-EUC0402
- removed C17: 10n, resistor:C-EUC0402
- removed C5: NF, resistor:C-EUC0402
- removed C6, C7: 10u, resistor:C-EUC0805
- removed C9: 100n, resistor:C-EUC0402
- removed F1: MF-MSMF200, openblw:MF-MSMF075/24
- removed IC1: V7805-1000, openblw:VR_1OUTXX
- removed K1: 61400416021, openblw:61400416021
- removed L1, L2: 4.7u, openblw:BOURNS-SRN4018
- removed L3: 10u, openblw:BOURNS-SRN4018
- removed PCB1: 1473005-4, openblw:RPI_COMPUTE
- removed R10, R7, R8, R9: 0R, resistor:R-EU_R0805
- removed R11, R12: 100K, resistor:R-EU_R0402
- removed R13, R14, R16, R17: 1.8K, resistor:R-EU_R0402
- removed R15, R6: 470R, resistor:R-EU_R0402
- removed R18: 1K, resistor:R-EU_R0402
- removed R4, R5: NR, resistor:R-EU_R0402
- removed U2: SFW15R-1STE1LF, openblw:RPI_CAMERA
- removed U3: DMG1012T, openblw:DMG1012T
- removed U4: TENDA_P200, openblw:TENDA_P200
- removed U5: PAM2306AYPKE, openblw:PAM2306
- removed U6: AP7115-25SEG, openblw:AP7115-XXSEG
- added FB2, FB3: (no value), openblw:FERRITESIZE_0805
- added Q1: (no value), openblw:NMOS-FETSOT23
- added U$1, U$2: ESC_POWER, openblw:ESC_POWER
- C2, C3: value 10u -> (none); device resistor:C-EUC0805 -> resistor:CPOL-EU153CLV-0810
- C4: value NF -> 10u
- CN1: value B2B-PH-K-S -> (none)
- FB1: value MI0805K601R-10 -> (none)
- JP1: value 90131-0764 -> (none); device pinhead:PINHD-2X4 -> pinhead:PINHD-1X4
- LED1: value RED -> LTW-5630AZL; device led:LEDCHIP-LED0603 -> openblw:LTW-5630AZL
- LED2: value GREEN -> LTW-5630AZL; device led:LEDCHIP-LED0603 -> openblw:LTW-5630AZL
- R1: value 100K -> 4.99K
- R2: value 0R -> 100K
- R3: value 0R -> 1K
- U1: value SFW15R-1STE1LF -> AL5812MP-13; device openblw:RPI_CAMERA -> openblw:AL5812MP-13
Connections:
- removed net +12V: C15.+, F1.2, IC1.IN
- removed net +1V8: C5.1, C7.1, L2.1, R3.1, R9.2
- removed net +2V5: C10.1, R10.2, U6.OUT@5
- removed net +3V3: C4.1, C6.1, C8.1, L1.1, R13.2, R14.2, R15.1, R16.2, R17.2, R2.1, R6.1, R7.2, R8.2, U1.CAM_3V3@15, U2.CAM_3V3@15, U4.3V3, U6.EN@3, U6.IN@1
- removed net +5V: C11.+, C2.1, C3.1, IC1.OUT, JP1.1, JP1.2, K1.VCC, R1.1, U5.EN1@6, U5.VIN1@7, U5.VIN2@1
- removed net BOTTOM_LIGHT_ENABLED: PCB1.59/GPIO17
- removed net CAM0_C_N: PCB1.144/CAM0_CN*, U1.CAM_CK_N@8
- removed net CAM0_C_P: PCB1.142/CAM0_CP*, U1.CAM_CK_P@9
- removed net CAM0_D0_N: PCB1.138/CAM0_DN0*, U1.CAM_D0_N@2
- removed net CAM0_D0_P: PCB1.136/CAM0_DP0*, U1.CAM_D0_P@3
- removed net CAM0_D1_N: PCB1.150/CAM0_DN1*, U1.CAM_D1_N@5
- removed net CAM0_D1_P: PCB1.148/CAM0_DP1*, U1.CAM_D1_P@6
- removed net CAM0_IO0: PCB1.36/GPIO31, U1.CAM_IO0@11
- removed net CAM0_IO1: PCB1.34/GPIO30, U1.CAM_IO1@12
- removed net CAM0_SCL: PCB1.30/GPIO29, R13.1, U1.CAM_SCL@13
- removed net CAM0_SDA: PCB1.28/GPIO28, R14.1, U1.CAM_SDA@14
- removed net CAM1_C_N: PCB1.149/CAM1_CN*, U2.CAM_CK_N@8
- removed net CAM1_C_P: PCB1.147/CAM1_CP*, U2.CAM_CK_P@9
- removed net CAM1_D0_N: PCB1.161/CAM1_DN0*, U2.CAM_D0_N@2
- removed net CAM1_D0_P: PCB1.159/CAM1_DP0*, U2.CAM_D0_P@3
- removed net CAM1_D1_N: PCB1.155/CAM1_DN1*, U2.CAM_D1_N@5
- removed net CAM1_D1_P: PCB1.153/CAM1_DP1*, U2.CAM_D1_P@6
- removed net CAM1_IO0: PCB1.11/GPIO3, U2.CAM_IO0@11
- removed net CAM1_IO1: PCB1.9/GPIO2, U2.CAM_IO1@12
- removed net CAM1_SCL: PCB1.5/GPIO1, R17.1, U2.CAM_SCL@13
- removed net CAM1_SDA: PCB1.3/GPIO0, R16.1, U2.CAM_SDA@14
- removed net CM_1V8: C12.1, PCB1.183/1V8, PCB1.184/1V8, PCB1.185/1V8, PCB1.186/1V8, R9.1
- removed net CM_3V3: C13.1, PCB1.191/3V3, PCB1.192/3V3, PCB1.193/3V3, PCB1.194/3V3, R8.1
- removed net CM_VBAT: C14.1, PCB1.197/VBAT, PCB1.198/VBAT, PCB1.199/VBAT, PCB1.200/VBAT, R7.1
- removed net CM_VDAC: PCB1.189/VDAC, PCB1.190/VDAC, R10.1
- removed net EMMC_DISABLE_N: PCB1.2/EMMC_DISABLE_N
- removed net EXT0/UART1_TX: JP1.6, PCB1.70/GPIO40
- removed net EXT1/UART1_RX: JP1.4, PCB1.72/GPIO41
- removed net GPIO47_1V8: PCB1.90/GPIO47_1V8, U3.G
- removed net N$10: C5.2, R3.2, R4.1, U5.FB2@10
- removed net N$11: PCB1.154/NC
- removed net N$12: PCB1.156/NC
- removed net N$13: PCB1.158/NC
- removed net N$14: PCB1.160/NC
- removed net N$15: PCB1.162/NC
- removed net N$16: PCB1.10/NC
- removed net N$17: PCB1.12/NC
- removed net N$18: PCB1.14/NC
- removed net N$19: PCB1.16/NC
- removed net N$20: PCB1.18/NC
- removed net N$21: PCB1.20/NC
- removed net N$22: PCB1.22/NC
- removed net N$23: PCB1.24/NC
- removed net N$24: PCB1.124/NC
- removed net N$25: PCB1.126/NC
- removed net N$26: PCB1.128/NC
- removed net N$27: PCB1.130/NC
- removed net N$28: PCB1.132/NC
- removed net N$29: PCB1.4/NC
- removed net N$30: PCB1.6/NC
- removed net N$31: PCB1.82/GPIO44, R12.1
- removed net N$32: LED2.A, R15.2
- removed net N$33: LED2.C, U3.D
- removed net N$34: PCB1.84/GPIO45, R11.1
- removed net N$35: PCB1.8/NC
- removed net N$36: CN1.2, FB1.1
- removed net N$37: C16.1, F1.1, L3.1
- removed net N$38: C17.1, R18.2
- removed net N$9: LED1.A, R6.2
- removed net PLC_N: U4.INN
- removed net PLC_P: U4.INP
- removed net TOP_LIGHT_ENABLED: PCB1.57/GPIO16
- removed net UART0_RX: JP1.5, PCB1.53/GPIO15
- removed net UART0_TX: JP1.3, PCB1.51/GPIO14
- removed net USB_D_N: K1.D-, PCB1.167/USB_DM**
- removed net USB_D_P: K1.D+, PCB1.165/USB_DP**
- new net LIGHT_PWM: JP1.1, R3.2
- new net VCC: CN1.1, FB1.1, FB2.1, FB3.1
- net GND: now also C1.1, C2.-, C3.-, C4.2, CN1.2, Q1.S, R2.1, U$1.GND, U$2.GND, U1.GND; no longer C1.2, C10.2, C11.-, C12.2, C13.2, C14.2, C15.-, C16.2, C17.2, C2.2, C3.2, C6.2, C7.2, C8.2, C9.2, CN1.1, IC1.GND, JP1.7, JP1.8, K1.GND, LED1.C, PCB1.1/GND, PCB1.103/GND, PCB1.104/GND, PCB1.109/GND, PCB1.110/GND, PCB1.115/GND, PCB1.121/GND, PCB1.122/GND, PCB1.127/GND, PCB1.13/GND, PCB1.133/GND, PCB1.134/GND, PCB1.139/GND, PCB1.140/GND, PCB1.145/GND, PCB1.146/GND, PCB1.151/GND, PCB1.152/GND, PCB1.157/GND, PCB1.163/GND, PCB1.164/GND, PCB1.169/GND, PCB1.170/GND, PCB1.181/GND, PCB1.182/GND, PCB1.187/GND, PCB1.188/GND, PCB1.19/GND, PCB1.195/GND, PCB1.196/GND, PCB1.25/GND, PCB1.26/GND, PCB1.31/GND, PCB1.32/GND, PCB1.37/GND, PCB1.38/GND, PCB1.43/GND, PCB1.44/GND, PCB1.49/GND, PCB1.50/GND, PCB1.55/GND, PCB1.56/GND, PCB1.61/GND, PCB1.62/GND, PCB1.67/GND, PCB1.68/GND, PCB1.7/GND, PCB1.73/GND, PCB1.74/GND, PCB1.79/GND, PCB1.80/GND, PCB1.85/GND, PCB1.86/GND, PCB1.91/GND, PCB1.92/GND, PCB1.97/GND, PCB1.98/GND, R11.2, R12.2, R4.2, R5.2, U1.CAM_GND@1, U1.CAM_GND@10, U1.CAM_GND@4, U1.CAM_GND@7, U2.CAM_GND@1, U2.CAM_GND@10, U2.CAM_GND@4, U2.CAM_GND@7, U3.S, U4.GND, U5.GND@3, U5.GND@9, U5.PAD, U6.GND@2
- net N$1: now also LED1.C, LED2.A; no longer C1.1, R1.2, U5.EN2@12
- net N$2: now also C1.2, LED2.C, U1.LED, U1.VCC; no longer L1.2, U5.LX1@8
- net N$3: now also C3.+, FB3.2, U$2.POWER; no longer U5.NC1@5
- net N$4: now also C4.1, FB1.2, LED1.A; no longer U5.NC2@11
- net N$5: now also R1.2, U1.RSET; no longer C9.1, U6.BP@4
- net N$6: now also Q1.D, R1.1; no longer FB1.2, L3.2, R18.1
- net N$7: now also Q1.G, R2.2, R3.1; no longer L2.2, U5.LX2@2
- net N$8: now also C2.+, FB2.2, U$1.POWER; no longer C4.2, R2.2, R5.1, U5.FB1@4
Other:
- note removed: "Camera"
- note removed: "Interfaces"
- note removed: "Power"
- note removed: "RPCM"
