File: pcb/main_controller_board/main_controller_board.brd (EAGLE design)
At the start: 72 x 50 mm, 58 parts, among them CN1 B2B-PH-K-S, IC1 V7805-1000, K1 61400416021, U1 SFW15R-1STE1LF, U2 SFW15R-1STE1LF, U3 DMG1012T, U4 TENDA_P200, U5 PAM2306AYPKE, U6 AP7115-25SEG

Commit message: fusion
Connections:
- net +3V3: now also PCB1.39, PCB1.40, PCB1.41, PCB1.42
Routing:
- net +3V3: track 160.9 -> 196.1 mm, vias 5 -> 9
Changed lines of the file:
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@@
 <via x="44.2849" y="21.6535" extent="1-16" drill="0.3"/>
 <via x="42.7609" y="19.3675" extent="1-16" drill="0.3"/>
-<via x="49.8729" y="17.5895" extent="1-16" drill="0.3"/>
-<via x="54.6989" y="21.9075" extent="1-16" drill="0.3"/>
+<via x="49.8729" y="17.5895" extent="1-16" drill="0.4"/>
+<via x="53.6829" y="20.6375" extent="1-16" drill="0.3"/>
 <via x="48.3489" y="20.8915" extent="1-16" drill="0.3"/>
 <via x="60.5409" y="21.6535" extent="1-16" drill="0.3"/>
-<via x="56.2229" y="17.3355" extent="1-16" drill="0.3"/>
+<via x="57.4929" y="17.5895" extent="1-16" drill="0.3"/>
 <via x="67.1449" y="21.6535" extent="1-16" drill="0.3"/>
 <via x="67.3989" y="17.5895" extent="1-16" drill="0.3"/>
@@
 <via x="45.5549" y="11.4935" extent="1-16" drill="0.3"/>
 <via x="47.5869" y="13.5255" extent="1-16" drill="0.3"/>
-<via x="51.3969" y="13.5255" extent="1-16" drill="0.3"/>
-<via x="49.8729" y="11.2395" extent="1-16" drill="0.3"/>
+<via x="51.6509" y="13.5255" extent="1-16" drill="0.3"/>
+<via x="49.3649" y="12.0015" extent="1-16" drill="0.3"/>
 <via x="55.4609" y="13.7795" extent="1-16" drill="0.3"/>
 <via x="58.2549" y="11.4935" extent="1-16" drill="0.3"/>
@@
 <wire x1="8.89" y1="3.81" x2="11.176" y2="1.524" width="0.8128" layer="15"/>
 <wire x1="11.176" y1="1.524" x2="35.052" y2="1.524" width="0.8128" layer="15"/>
-<wire x1="35.052" y1="1.524" x2="61.722" y2="1.524" width="0.8128" layer="15"/>
+<wire x1="35.052" y1="1.524" x2="50.546" y2="1.524" width="0.8128" layer="15"/>
+<wire x1="50.546" y1="1.524" x2="61.722" y2="1.524" width="0.8128" layer="15"/>
 <wire x1="62.118" y1="2.794" x2="62.118" y2="1.92" width="0.4064" layer="1"/>
 <wire x1="62.118" y1="1.92" x2="61.722" y2="1.524" width="0.4064" layer="1"/>
@@
 <via x="35.052" y="1.524" extent="1-16" drill="0.4"/>
 <wire x1="35.4584" y1="2.7836" x2="35.448" y2="2.794" width="0.4064" layer="1"/>
+<contactref element="PCB1" pad="42"/>
+<contactref element="PCB1" pad="40"/>
+<contactref element="PCB1" pad="39"/>
+<contactref element="PCB1" pad="41"/>
+<via x="52.07" y="17.018" extent="1-16" drill="0.4"/>
+<wire x1="52.07" y1="17.018" x2="50.546" y2="15.494" width="0.8128" layer="15"/>
+<wire x1="50.546" y1="15.494" x2="50.546" y2="1.524" width="0.8128" layer="15"/>
+<wire x1="56.175" y1="15.458" x2="56.175" y2="16.805" width="0.254" layer="16"/>
+<wire x1="56.175" y1="16.805" x2="56.134" y2="17.018" width="0.254" layer="16"/>
+<via x="56.134" y="17.018" extent="1-16" drill="0.4"/>
+<wire x1="56.134" y1="17.018" x2="52.07" y2="17.018" width="0.8128" layer="15"/>
+<wire x1="51.975" y1="15.458" x2="51.975" y2="16.923" width="0.254" layer="16"/>
+<wire x1="51.975" y1="16.923" x2="52.07" y2="17.018" width="0.254" layer="16"/>
+<wire x1="55.875" y1="23.658" x2="55.875" y2="22.601" width="0.254" layer="16"/>
+<wire x1="55.875" y1="22.601" x2="55.372" y2="22.098" width="0.254" layer="16"/>
+<via x="55.372" y="22.098" extent="1-16" drill="0.4"/>
+<wire x1="55.372" y1="22.098" x2="52.07" y2="22.098" width="0.8128" layer="15"/>
+<via x="52.07" y="22.098" extent="1-16" drill="0.4"/>
+<wire x1="52.07" y1="22.098" x2="51.675" y2="22.493" width="0.254" layer="16"/>
+<wire x1="51.675" y1="22.493" x2="51.675" y2="23.658" width="0.254" layer="16"/>
+<wire x1="52.07" y1="22.098" x2="52.07" y2="17.018" width="0.8128" layer="15"/>
 </signal>
 <signal name="+1V8">
