File: pcb/main_controller_board/main_controller_board.sch (EAGLE design)
At the start: 57 parts, among them CN1 B2B-PH-K-S, IC1 V7805-1000, K1 61400416021, U1 SFW15R-1STE1LF, U2 SFW15R-1STE1LF, U3 DMG1012T, U4 TENDA_P200, U5 PAM2306AYPKE, U6 AP7115-25SEG

Commit message: fusion
Connections:
- net +3V3: now also PCB1.39/GPIO0-27_VREF, PCB1.40/GPIO0-27_VREF, PCB1.41/GPIO28-45_VREF, PCB1.42/GPIO28-45_VREF
Changed lines of the file:
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@@
 <part name="GND26" library="supply" deviceset="GND" device=""/>
 <part name="GND30" library="supply" deviceset="GND" device=""/>
+<part name="V33" library="supply" deviceset="+3V3" device=""/>
+<part name="V35" library="supply" deviceset="+3V3" device=""/>
 </parts>
 <sheets>
@@
 <instance part="V29" gate="G$1" x="45.72" y="78.74"/>
 <instance part="V30" gate="G$1" x="157.48" y="78.74"/>
+<instance part="V33" gate="G$1" x="228.6" y="309.88" rot="R270"/>
+<instance part="V35" gate="G$1" x="50.8" y="309.88" rot="R90"/>
 </instances>
 <busses>
@@
 <wire x1="45.72" y1="48.26" x2="55.88" y2="48.26" width="0.1524" layer="91"/>
 </segment>
-</net>
+<segment>
+<pinref part="PCB1" gate="G$1" pin="42/GPIO28-45_VREF"/>
+<wire x1="177.8" y1="309.88" x2="226.06" y2="309.88" width="0.1524" layer="91"/>
+<pinref part="V33" gate="G$1" pin="+3V3"/>
+<pinref part="PCB1" gate="G$1" pin="40/GPIO0-27_VREF"/>
+<wire x1="177.8" y1="312.42" x2="226.06" y2="312.42" width="0.1524" layer="91"/>
+<wire x1="226.06" y1="312.42" x2="226.06" y2="309.88" width="0.1524" layer="91"/>
+<junction x="226.06" y="309.88"/>
+</segment>
+<segment>
+<pinref part="V35" gate="G$1" pin="+3V3"/>
+<pinref part="PCB1" gate="G$1" pin="39/GPIO0-27_VREF"/>
+<wire x1="76.2" y1="312.42" x2="53.34" y2="312.42" width="0.1524" layer="91"/>
+<wire x1="53.34" y1="312.42" x2="53.34" y2="309.88" width="0.1524" layer="91"/>
+<junction x="53.34" y="309.88"/>
+<pinref part="PCB1" gate="G$1" pin="41/GPIO28-45_VREF"/>
+<wire x1="53.34" y1="309.88" x2="76.2" y2="309.88" width="0.1524" layer="91"/>
+</segment>
+</net>
