File: pcb/driver_board/driver_board.brd (EAGLE design)
At the start: 65 x 56 mm, 22 parts, among them U1 AL5812MP-13

Commit message: client board
Parts:
- removed C4: 10u, resistor:C0402
- removed CN1: (no value), openblw:JST-PH-2-THM
- removed FB1, FB2, FB3: (no value), openblw:R0805
- added ESC1: ESC_POWER, openblw:ESC_POWER
- added LOGO1: (no value), openblw:OHMYDIGIFAB_LOGO
- U$1: value ESC_POWER -> 282836-2; device openblw:ESC_POWER -> openblw:282836-2
- moved U$1 52.9 mm to (14.0, 52.1), turned to 0 degrees
- moved JP1 23.1 mm to (51.4, 3.81), turned to 180 degrees
- moved C1 9.83 mm to (45.9, 22.2)
- moved LED1 3.00 mm to (17.0, 28.0)
- moved LED2 3.00 mm to (48.0, 28.0)
- moved Q1 2.54 mm to (50.8, 14.0)
- moved R1 2.54 mm to (47.0, 14.0)
- moved U1 2.54 mm to (48.3, 19.1)
- moved C3 1.27 mm to (52.1, 48.3)
- moved R2 1.27 mm to (54.6, 12.7)
- moved R3 1.27 mm to (54.6, 10.2)
- renumbered U$2 to ESC2
Connections:
- removed net N$2: C1.2, LED2.C1, LED2.C2, U1.1, U1.8
- removed net N$3: C3.+, ESC2.PWR1, ESC2.PWR2, FB3.2
- removed net N$4: C4.1, FB1.2, LED1.A1, LED1.A2, LED1.A3
- removed net N$8: C2.+, FB2.2, U$1.PWR1, U$1.PWR2
- new net N$9: LED2.C1, LED2.C2, U1.8
- net GND: now also ESC1.GND1, ESC1.GND2, U$1.CON2, U1.HSINK; no longer C4.2, CN1.1, U$1.GND1, U$1.GND2
- net VCC: now also C1.2, C2.+, C3.+, ESC1.PWR1, ESC1.PWR2, ESC2.PWR1, ESC2.PWR2, LED1.A1, LED1.A2, LED1.A3, U$1.CON1, U1.1; no longer CN1.2, FB1.1, FB2.1, FB3.1
Routing:
- net N$4: track 17.7 -> 0.00 mm
- net N$2: track 17.6 -> 0.00 mm
- net N$8: track 16.6 -> 0.00 mm
- net N$3: track 13.7 -> 0.00 mm
- net LIGHT_PWM: track 15.4 -> 6.36 mm
- net N$9: track 0.00 -> 8.69 mm
- net VCC: track 75.8 -> 82.9 mm, vias 0 -> 1
- net N$1: track 40.7 -> 43.4 mm
- net N$7: track 6.00 -> 4.73 mm
- added copper zone on layer 16, net VCC
Other:
- outline, holes or cut-outs redrawn
- board text added: "Driver Board"
- board text added: "OpenBLW"
- board text added: "Rev.0.1"

Commit message: before order pcbs
Parts:
- C2, C3: value (none) -> UWT1E221MNL1GS(220u)
- JP1: value (none) -> M20-9990446
- LED1, LED2: value LTW-5630AZL -> LTW-5630AZL50
- Q1: value (none) -> IRLML6346TRPBF
Other:
- board text added: "VCC"
Changed lines of the file:
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@@
 <text x="59.309" y="19.05" size="1.6764" layer="21" rot="R90">Driver Board</text>
 <text x="61.849" y="19.05" size="1.4224" layer="21" rot="R90">Rev.0.1</text>
+<text x="9.525" y="46.101" size="1.4224" layer="21">VCC</text>
 </plain>
 <attributes>
@@
 </autorouter>
 <elements>
-<element name="Q1" library="openblw" package="SOT23" value="" x="50.8" y="13.97" smashed="yes" rot="R90">
+<element name="Q1" library="openblw" package="SOT23" value="IRLML6346TRPBF" x="50.8" y="13.97" smashed="yes" rot="R90">
 <attribute name="NAME" x="54.045" y="14.69" size="1.016" layer="25" font="vector" ratio="10" rot="R90"/>
 </element>
@@
 <attribute name="NAME" x="46.99" y="15.875" size="1.016" layer="25" font="vector" ratio="10"/>
 </element>
-<element name="LED1" library="openblw" package="LITEON-5630" value="LTW-5630AZL" x="17" y="28" smashed="yes" rot="R180">
+<element name="LED1" library="openblw" package="LITEON-5630" value="LTW-5630AZL50" x="17" y="28" smashed="yes" rot="R180">
 <attribute name="NAME" x="19.065" y="25.9" size="1.016" layer="25" font="vector" ratio="10" rot="R180"/>
 </element>
-<element name="LED2" library="openblw" package="LITEON-5630" value="LTW-5630AZL" x="48" y="28" smashed="yes" rot="R180">
+<element name="LED2" library="openblw" package="LITEON-5630" value="LTW-5630AZL50" x="48" y="28" smashed="yes" rot="R180">
 <attribute name="NAME" x="50.065" y="25.9" size="1.016" layer="25" font="vector" ratio="10" rot="R180"/>
 </element>
@@
 <attribute name="NAME" x="33.77" y="50.025" size="1.016" layer="25" font="vector" ratio="10" rot="R180"/>
 </element>
-<element name="C2" library="resistor" package="153CLV-0810" value="" x="12.7" y="7.62" smashed="yes">
+<element name="C2" library="resistor" package="153CLV-0810" value="UWT1E221MNL1GS(220u)" x="12.7" y="7.62" smashed="yes">
 <attribute name="NAME" x="8.41" y="12.15" size="1.016" layer="25"/>
 <attribute name="VALUE" x="8.375" y="1.835" size="1.27" layer="27"/>
 </element>
-<element name="C3" library="resistor" package="153CLV-0810" value="" x="52.07" y="48.26" smashed="yes" rot="R180">
+<element name="C3" library="resistor" package="153CLV-0810" value="UWT1E221MNL1GS(220u)" x="52.07" y="48.26" smashed="yes" rot="R180">
 <attribute name="NAME" x="56.36" y="43.73" size="1.016" layer="25" rot="R180"/>
 <attribute name="VALUE" x="56.395" y="54.045" size="1.27" layer="27" rot="R180"/>
@@
 <element name="H3" library="holes" package="2,8-PAD" value="MOUNT-PAD-ROUND2.8" x="3.6" y="52.4" smashed="yes"/>
 <element name="H4" library="holes" package="2,8-PAD" value="MOUNT-PAD-ROUND2.8" x="61.4" y="52.4" smashed="yes"/>
-<element name="JP1" library="pinhead" package="1X04" value="" x="51.435" y="3.81" smashed="yes" rot="R180">
+<element name="JP1" library="pinhead" package="1X04" value="M20-9990446" x="51.435" y="3.81" smashed="yes" rot="R180">
 <attribute name="NAME" x="56.5912" y="1.9812" size="1.016" layer="25" ratio="10" rot="R180"/>
 <attribute name="VALUE" x="56.515" y="6.985" size="1.27" layer="27" rot="R180"/>

Commit message: ordered
Parts:
- moved C1 1.27 mm to (44.7, 22.2)
- moved U$1 0.63 mm to (14.6, 52.1)
Routing:
- net VCC: track 82.9 -> 77.2 mm, vias 1 -> 0
- net N$1: track 43.4 -> 38.5 mm
- added copper zone on layer 1, net VCC
- removed copper zone on layer 16, net VCC
