File: pcb/client_board/client_board.brd (EAGLE design)
At the start: 65 x 56 mm, 20 parts, among them IC1 V7805-1000, J2 PJ-102AH/BH, J3 RASPBERRYPI-40-PIN-GPIO, U4 TENDA_P200

Commit message: before order pcbs
Parts:
- removed R1, R2: 0R, resistor:R0603
- removed U4: TENDA_P200, openblw:TENDA_P200
- added FB2: MI0805K601R-10, resistor:L5650M
- added JP2, JP3: M20-9980346, pinhead:2X03
- added U$2: (no value), openblw:TENDA_P200
- C11: value 22u -> UUD1A220MCL1GS(22u)
- C15: value 10u -> UUD1E100MCL1GS(10u)
- C16: value 1u -> EMK105BJ105KV-F(1u)
- C17: value 10n -> EMK105B7103KV-F(10n)
- F1: value MF-MSMF200 -> MF-MSMF200-2
- J2: value PJ-102AH/BH -> PJ-102AH
- J3: value RASPBERRYPI-40-PIN-GPIO -> SFH11-PBPC-D20-ST-BK
- L3: value SRP1250-100M -> SRP1245A-100M; device openblw:SRP1250 -> openblw:SRP1250A
- R18: value 1K -> ERJ-2GEJ102X(1K)
- moved FB1 44.3 mm to (61.0, 21.6), turned to 270 degrees
- moved U$1 43.7 mm to (57.1, 12.7)
- moved C17 39.7 mm to (59.7, 44.0), turned to 90 degrees
- moved C16 37.5 mm to (47.6, 28.8), turned to 270 degrees
- moved J2 36.8 mm to (52.1, 45.7)
- moved L3 36.5 mm to (56.5, 33.0)
- moved R18 35.9 mm to (59.7, 41.6), turned to 90 degrees
- moved LOGO1 35.5 mm to (23.4, 40.9), turned to 0 degrees
- moved IC1 33.8 mm to (39.4, 38.7), turned to 270 degrees
- moved F1 33.4 mm to (45.1, 38.7), turned to 180 degrees
- moved C15 30.1 mm to (30.5, 41.3)
- moved C11 21.3 mm to (30.5, 36.2), turned to 0 degrees
Connections:
- removed net AVCC_: FB1.2, U$1.CON1
- removed net PLC_N: R2.1, U4.5, U4.6
- removed net PLC_P: R1.2, U4.1, U4.2
- net +3V3: now also JP3.5, JP3.6; no longer U4.7, U4.8
- net AGND: now also FB2.2, JP2.5, JP2.6, U$1.CON1; no longer R2.2
- net AVCC: now also FB1.2, JP2.1, JP2.2, U$1.CON2; no longer R1.1
- net GND: now also FB2.1, JP3.1; no longer U$1.CON2, U4.12
Routing:
- net PLC_P: track 53.9 -> 0.00 mm
- net PLC_N: track 53.1 -> 0.00 mm
- net AVCC_: track 16.8 -> 0.00 mm
- net +12V: track 36.9 -> 21.7 mm
- net AVCC: track 5.13 -> 15.0 mm
- net N$9: track 31.8 -> 22.7 mm
- net +3V3: track 28.1 -> 34.6 mm
- net GND: track 0.00 -> 5.19 mm, vias 96 -> 90
- net AGND: track 5.13 -> 10.0 mm
- net +5V: track 57.2 -> 54.2 mm
- net N$38: track 1.88 -> 1.04 mm
- added copper zone on layer 16, net +5V
- added copper zone on layer 1, net AGND
- added copper zone on layer 1, net AVCC
- removed copper zone on layer 1, net AVCC_
Other:
- board text added: "VCC"

Commit message: parts miss
Parts:
- FB1, FB2: value MI0805K601R-10 -> HR2220V801R-10
Changed lines of the file:
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@@
 <attribute name="VALUE" x="28.205" y="37.54" size="1.27" layer="27" display="off"/>
 </element>
-<element name="FB1" library="resistor" package="L5650M" value="MI0805K601R-10" x="60.96" y="21.59" smashed="yes" rot="R270">
+<element name="FB1" library="resistor" package="L5650M" value="HR2220V801R-10" x="60.96" y="21.59" smashed="yes" rot="R270">
 <attribute name="NAME" x="56.515" y="20.32" size="1.27" layer="25" rot="R270"/>
 <attribute name="VALUE" x="56.515" y="23.495" size="1.27" layer="27" rot="R270" display="off"/>
@@
 </element>
 <element name="LOGO1" library="openblw" package="OHMYDIGIFAB_LOGO" value="" x="23.368" y="40.894" smashed="yes"/>
-<element name="FB2" library="resistor" package="L5650M" value="MI0805K601R-10" x="53.34" y="21.59" smashed="yes" rot="R270">
+<element name="FB2" library="resistor" package="L5650M" value="HR2220V801R-10" x="53.34" y="21.59" smashed="yes" rot="R270">
 <attribute name="NAME" x="49.53" y="20.32" size="1.27" layer="25" rot="R270"/>
 <attribute name="VALUE" x="48.895" y="23.495" size="1.27" layer="27" rot="R270" display="off"/>

Commit message: ordered
Parts:
- moved C17 20.0 mm to (46.9, 28.6), turned to 180 degrees
- moved R18 16.3 mm to (49.8, 28.6), turned to 180 degrees
- moved C16 9.40 mm to (49.0, 38.1)
- moved L3 2.84 mm to (57.8, 35.6), turned to 180 degrees
- moved F1 2.54 mm to (45.1, 41.3)
Routing:
- net N$9: track 22.7 -> 19.6 mm
- net +12V: track 21.7 -> 19.7 mm
- net N$4: track 11.7 -> 10.6 mm
- net N$38: track 1.04 -> 1.67 mm
- net GND: vias 90 -> 92
