File: pcb/interface_board/interface_board.brd (EAGLE design)
At the start: 72 x 50 mm, 58 parts, among them CN1 B2B-PH-K-S, IC1 V7805-1000, K1 61400416021, U1 SFW15R-1STE1LF, U2 SFW15R-1STE1LF, U3 DMG1012T, U4 TENDA_P200, U5 PAM2306AYPKE, U6 AP7115-25SEG

Commit message: client board
Parts:
- removed C10: 4.7u, resistor:C0603
- removed C8: 1u, resistor:C0402
- removed C9: 100n, resistor:C0402
- removed CN1: B2B-PH-K-S, openblw:JST-PH-2-THM
- removed R10: 0R, resistor:R0805
- removed U6: AP7115-25SEG, openblw:SOT353
- added U$1, U$2: 282836-2, openblw:282836-2
- FB1: device openblw:R0805 -> resistor:L5650M
- L3: device openblw:BOURNS-SRN4018 -> openblw:SRP1250
- moved JP1 41.4 mm to (59.9, 11.4), flipped to the top
- moved LOGO1 38.6 mm to (39.6, 11.7)
- moved C15 26.4 mm to (40.3, 28.4)
- moved U4 19.5 mm to (22.1, 50.0)
- moved C17 18.4 mm to (11.9, 30.2), turned to 270 degrees
- moved R18 17.8 mm to (10.7, 31.5), turned to 270 degrees
- moved C11 17.7 mm to (32.8, 28.4), turned to 180 degrees
- moved FB1 14.9 mm to (11.2, 37.6), turned to 270 degrees
- moved C16 12.1 mm to (33.3, 40.6)
- moved IC1 11.9 mm to (36.6, 30.5)
- moved K1 8.89 mm to (45.5, 39.6)
- moved F1 8.59 mm to (33.4, 38.0), turned to 0 degrees
- moved L3 7.47 mm to (21.8, 35.1), turned to 270 degrees
- moved R9 6.28 mm to (9.14, 26.9)
- moved C1 6.14 mm to (17.5, 41.1), flipped to the bottom
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Connections:
- removed net +2V5: C10.1, R10.2, U6.5
- removed net CM_VDAC: PCB1.189, PCB1.190, R10.1
- removed net N$37: C16.1, F1.1, L3.P$1
- removed net N$5: C9.1, U6.4
- new net N$39: C15.+, F1.2, IC1.IN
- net +12V: now also C16.1, F1.1, L3.1, U$2.CON1; no longer C15.+, F1.2, IC1.IN
- net +3V3: no longer C8.1, PCB1.39, PCB1.40, PCB1.41, PCB1.42, U6.1, U6.3
- net +5V: now also PCB1.39, PCB1.40, PCB1.41, PCB1.42
- net CM_3V3: now also PCB1.189, PCB1.190
- net GND: now also U$1.CON2, U$2.CON2; no longer C10.2, C8.2, C9.2, CN1.2, U6.2
- net N$36: now also U$1.CON1; no longer CN1.1
- net N$6: now also L3.2; no longer L3.P$2
Routing:
- net +5V: track 67.0 -> 118.0 mm, vias 3 -> 8
- net PLC_N: track 36.5 -> 6.37 mm
- net +2V5: track 19.3 -> 0.00 mm
- net CM_VDAC: track 17.6 -> 0.00 mm
- net UART0_TX: track 31.7 -> 14.1 mm
- net PLC_P: track 28.1 -> 11.7 mm
- net UART0_RX: track 33.0 -> 16.8 mm
- net +3V3: track 196.1 -> 210.3 mm, vias 9 -> 4
- net N$39: track 0.00 -> 12.3 mm
- net +12V: track 12.1 -> 0.00 mm
- net +1V8: track 31.4 -> 42.6 mm
- net GND: track 25.3 -> 35.7 mm, vias 165 -> 138
- net GPIO47_1V8: track 43.6 -> 51.5 mm
- net CM_VBAT: track 22.4 -> 14.5 mm
- net CM_1V8: track 21.3 -> 14.1 mm
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- added copper zone on layer 1, net +12V
- added copper zone on layer 1, net N$36
- added copper zone on layer 1, net N$6
Other:
- board text added: "Interface Board"
- board text added: "Rev.0.3"
- board text removed: "MainController"
- board text removed: "Rev.0.2"

Commit message: 0.4
Parts:
- moved U4 58.5 mm to (61.2, 6.60), turned to 90 degrees
- moved C17 53.9 mm to (65.8, 28.4), turned to 0 degrees
- moved R18 52.2 mm to (62.7, 28.4), turned to 0 degrees
- moved U$1 49.3 mm to (64.5, 34.5), turned to 270 degrees
- moved FB1 46.1 mm to (57.1, 34.3)
- moved L3 37.7 mm to (56.9, 21.1), turned to 90 degrees
- moved U$2 31.8 mm to (64.5, 44.7), turned to 270 degrees
- moved C16 27.8 mm to (47.8, 17.0), turned to 270 degrees
- moved JP1 25.3 mm to (42.9, 30.1), turned to 90 degrees
- moved C11 25.2 mm to (7.84, 24.9), turned to 0 degrees
- moved F1 21.1 mm to (45.6, 20.9), turned to 180 degrees
- moved IC1 20.9 mm to (16.5, 24.6)
- moved C15 17.5 mm to (22.9, 29.0), turned to 270 degrees
- moved K1 9.47 mm to (36.0, 39.6)
- moved R13 8.27 mm to (53.2, 2.29), flipped to the bottom, turned to 270 degrees
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Routing:
- net +3V3: track 210.3 -> 180.4 mm
- net UART0_RX: track 16.8 -> 37.6 mm
- net UART0_TX: track 14.1 -> 35.0 mm
- net N$39: track 12.3 -> 30.9 mm, vias 0 -> 1
- net USB_D_N: track 51.3 -> 39.1 mm
- net USB_D_P: track 57.4 -> 45.2 mm
- net CAM1_SCL: track 61.6 -> 51.5 mm, vias 3 -> 2
- net PLC_P: track 11.7 -> 2.54 mm
- net GPIO47_1V8: track 51.5 -> 42.5 mm
- net CAM1_SDA: track 58.3 -> 50.8 mm, vias 3 -> 2
- net CAM0_SCL: track 30.3 -> 23.1 mm, vias 3 -> 2
- net CAM1_IO0: track 51.6 -> 46.0 mm
- net +5V: track 118.0 -> 112.8 mm, vias 8 -> 7
- net CAM0_SDA: track 27.9 -> 22.8 mm, vias 3 -> 2
- net GND: track 35.7 -> 40.2 mm, vias 138 -> 0
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- added copper zone on layer 16, net +12V
Other:
- board size 72 x 50 mm -> 72 x 56 mm

Commit message: rj45
Parts:
- added ETH1: HR911105A, openblw:RJ45
- L3: value 10u -> SRP1250A; device openblw:SRP1250 -> openblw:SRP1250A
- moved JP1 39.7 mm to (8.13, 11.0), turned to 0 degrees
- moved C15 19.8 mm to (3.17, 27.0)
- moved K1 9.19 mm to (29.0, 45.6)
- moved C11 2.08 mm to (8.00, 27.0), turned to 270 degrees
- moved L3 0.18 mm to (56.8, 21.0), turned to 270 degrees
Connections:
- net +12V: now also L3.2; no longer L3.1
- net N$6: now also L3.1; no longer L3.2
Routing:
- net +5V: track 112.8 -> 154.6 mm
- net EXT1/UART1_RX: track 20.0 -> 47.7 mm
- net EXT0/UART1_TX: track 23.9 -> 45.1 mm
- net GPIO47_1V8: track 42.5 -> 61.4 mm
- net UART0_TX: track 35.0 -> 51.5 mm
- net N$39: track 30.9 -> 46.6 mm
- net +1V8: track 42.6 -> 55.9 mm
- net UART0_RX: track 37.6 -> 50.5 mm
- net +3V3: track 180.4 -> 189.9 mm
- net USB_D_P: track 45.2 -> 38.0 mm
- net CAM0_D0_N: track 40.2 -> 46.8 mm
- net CAM0_D0_P: track 40.2 -> 46.7 mm
- net USB_D_N: track 39.1 -> 43.3 mm

Commit message: tune
Parts:
- moved LED2 20.9 mm to (5.84, 18.0), turned to 270 degrees
- moved R15 20.8 mm to (2.92, 18.0), turned to 0 degrees
- moved LED1 20.4 mm to (5.84, 20.1), turned to 270 degrees
- moved R6 20.3 mm to (2.92, 20.1), turned to 0 degrees
- moved U3 19.9 mm to (5.61, 16.1), turned to 0 degrees
- moved C14 8.19 mm to (13.3, 21.1), turned to 0 degrees
- moved C13 5.61 mm to (13.3, 19.1), turned to 0 degrees
- moved C12 3.51 mm to (13.3, 17.0), turned to 0 degrees
Routing:
- net GPIO47_1V8: track 61.4 -> 39.2 mm
- net CM_VBAT: track 14.5 -> 19.0 mm
- net CM_3V3: track 16.0 -> 18.1 mm
- net N$33: track 2.80 -> 1.92 mm
- net N$9: track 2.16 -> 1.52 mm
- net N$32: track 2.16 -> 1.52 mm
- net USB_D_N: track 43.3 -> 42.7 mm
- net USB_D_P: track 38.0 -> 37.5 mm
- net +3V3: track 189.9 -> 189.8 mm, vias 4 -> 6
- net GND: track 40.2 -> 40.3 mm, vias 0 -> 1

Commit message: tochu
Parts:
- moved R5 20.8 mm to (2.41, 47.8), turned to 270 degrees
- moved C4 19.0 mm to (3.81, 47.8), turned to 90 degrees
- moved C6 17.9 mm to (13.5, 54.2), turned to 0 degrees
- moved R2 17.1 mm to (5.21, 47.8), turned to 90 degrees
- moved L2 16.5 mm to (8.64, 45.6), turned to 90 degrees
- moved C2 15.5 mm to (13.5, 52.2), turned to 0 degrees
- moved L1 13.5 mm to (18.8, 53.0), turned to 270 degrees
- moved U5 11.9 mm to (13.7, 48.9), turned to 90 degrees
- moved C3 9.79 mm to (13.7, 46.1), turned to 180 degrees
- moved C7 9.11 mm to (13.7, 44.1), turned to 180 degrees
- moved R3 8.37 mm to (17.9, 48.9), turned to 90 degrees
- moved C5 7.86 mm to (19.2, 48.9), turned to 90 degrees
- moved R4 7.73 mm to (20.4, 48.9), turned to 270 degrees
- moved R1 4.79 mm to (17.8, 45.6), turned to 0 degrees
- moved C1 2.93 mm to (17.8, 44.1), turned to 180 degrees
Routing:
- net USB_D_N: track 42.7 -> 7.78 mm
- net USB_D_P: track 37.5 -> 7.77 mm
- net +1V8: track 55.9 -> 45.5 mm, vias 3 -> 2
- net +5V: track 154.6 -> 145.3 mm
- net +3V3: track 189.8 -> 194.6 mm, vias 6 -> 8
- net N$8: track 5.71 -> 9.98 mm
- net N$1: track 4.82 -> 6.34 mm
- net GND: track 40.3 -> 41.8 mm, vias 1 -> 3
- net N$5: track 1.01 -> 0.00 mm

Commit message: lan
Parts:
- removed ETH1: HR911105A, openblw:RJ45
- added C10, C41: 10u, rcl:C0805
- added C21, C22, C23, C24: 20p, rcl:C0603
- added C26, C27, C28, C29, C30, C31, C32, C33, C34, C35, C36, C37, C38, C39, C40, C43, C8, C9: 100n, rcl:C0603
- added C42: 1u, rcl:C0805
- added ETHERNET: HR911105A, hanrun:RJ45
- added FB2, FB3: FERRITE_BEAD, raspi:C0805
- added FB4: MI0805K601R-10, resistor:L5650M
- added IC6: LAN9512, raspi:QFN64-9X9
- added JP2, JP3: (no value), pinhead:1X01
- added R10, R20, R32, R37: 12k, rcl:R0603
- added R25, R26: 1k, rcl:R0603
- added R27: 10, rcl:R0603
- added R28, R29, R30, R31: 49.9, rcl:R0603
- added R33: 12k4, rcl:R0603
- moved C15 38.9 mm to (42.1, 26.3), turned to 180 degrees
- moved C11 34.4 mm to (42.1, 31.4), turned to 180 degrees
- moved C16 27.9 mm to (60.4, 41.9), turned to 90 degrees
- moved U$1 23.3 mm to (66.7, 11.3), turned to 0 degrees
- moved FB1 18.5 mm to (68.1, 19.3), turned to 90 degrees
- moved IC1 17.9 mm to (33.9, 28.8), turned to 90 degrees
- moved L3 14.7 mm to (65.4, 32.9), turned to 180 degrees
- moved F1 14.6 mm to (56.6, 30.7), turned to 270 degrees
- moved C17 10.0 mm to (56.1, 25.8), turned to 180 degrees
- moved R18 4.44 mm to (59.2, 25.8), turned to 180 degrees
- moved K1 3.88 mm to (32.9, 45.7)
- moved LOGO1 3.33 mm to (42.8, 12.7)
- moved U$2 2.54 mm to (67.1, 44.7), turned to 180 degrees
- moved C14 0.89 mm to (13.3, 22.0)
- moved LED1 0.76 mm to (5.84, 20.8)
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Connections:
- removed net N$36: FB1.1, U$1.CON1
- removed net PLC_N: U4.5, U4.6
- removed net PLC_P: U4.1, U4.2
- new net 3V3A: C8.1, C9.1, R27.1, R28.1, R29.1, R30.1, R31.1
- new net 3V3A1: C32.2, C33.2, C34.2, C35.2, C36.2, C37.2, C38.2, FB2.1, IC6.10, IC6.49, IC6.5, IC6.51, IC6.54, IC6.57, IC6.64
- new net AGND: FB4.1, U$1.CON1, U4.5, U4.6
- new net AVCC: FB1.1, U$1.CON2, U4.1, U4.2
- new net GPIO6: IC6.12, R37.2
- new net N$37: ETHERNET.12, R25.2
- new net N$40: ETHERNET.9, R26.2
- new net N$41: C26.1, ETHERNET.4, ETHERNET.5, R27.2
- new net N$42: IC6.63, R10.2
- new net N$43: C42.2, FB3.2, IC6.62
- new net N$44: IC6.41, R32.1
- new net N$45: IC6.50, R33.1
- new net N$46: IC6.28, R20.1
- new net NLNKA_LED: ETHERNET.10, IC6.21
- new net NSPD_LED: ETHERNET.11, IC6.22
- new net RX_N: C24.1, ETHERNET.6, IC6.53, R28.2
- new net RX_P: C23.1, ETHERNET.3, IC6.52, R29.2
- new net TX_N: C22.1, ETHERNET.2, IC6.56, R30.2
- new net TX_P: C21.1, ETHERNET.1, IC6.55, R31.2
- new net USBD3_N: IC6.3, K1.2
- new net USBD3_P: IC6.4, K1.3
- new net VDD18CORE: C39.2, C40.2, C41.2, IC6.15, IC6.38
- new net VDD18PLL: C43.2, FB3.1, IC6.48
- new net XI: IC6.61
- new net XO: IC6.60
- net +3V3: now also C27.1, C28.1, C29.1, C30.2, C31.2, FB2.2, IC6.11, IC6.19, IC6.27, IC6.33, IC6.39, IC6.40, IC6.46, JP2.1, R20.2, R25.1, R26.1, R32.2, R37.1
- net +5V: now also C10.1
- net GND: now also C10.2, C21.2, C22.2, C23.2, C24.2, C26.2, C27.2, C28.2, C29.2, C30.1, C31.1, C32.1, C33.1, C34.1, C35.1, C36.1, C37.1, C38.1, C39.1, C40.1, C41.1, C42.1, C43.1, C8.2, C9.2, ETHERNET.8, FB4.2, IC6.34, IC6.44, IC6.EXP, JP3.1, R10.1, R33.2; no longer U$1.CON2
- net USB_D_N: now also IC6.58; no longer K1.2
- net USB_D_P: now also IC6.59; no longer K1.3
Routing:
- net +3V3: track 194.6 -> 295.2 mm, vias 8 -> 17
- net 3V3A1: track 0.00 -> 66.8 mm, vias 0 -> 7
- net TX_N: track 0.00 -> 63.4 mm
- net RX_P: track 0.00 -> 59.1 mm
- net TX_P: track 0.00 -> 58.1 mm
- net RX_N: track 0.00 -> 56.0 mm
- net NLNKA_LED: track 0.00 -> 45.3 mm, vias 0 -> 1
- net NSPD_LED: track 0.00 -> 38.1 mm, vias 0 -> 1
- net VDD18CORE: track 0.00 -> 29.7 mm, vias 0 -> 2
- net N$39: track 46.5 -> 21.9 mm, vias 1 -> 0
- net USBD3_N: track 0.00 -> 22.1 mm
- net USBD3_P: track 0.00 -> 21.5 mm
- net N$43: track 0.00 -> 19.0 mm, vias 0 -> 2
- net +12V: track 0.00 -> 13.7 mm, vias 21 -> 0
- net AVCC: track 0.00 -> 13.2 mm
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- added copper zone on layer 1, net AGND
- added copper zone on layer 1, net AVCC
- removed copper zone on layer 16, net +12V
- removed copper zone on layer 1, net N$36
Other:
- outline, holes or cut-outs redrawn
- board text added: "3V3"
- board text added: "AVCC"
- board text added: "GND"
- board text added: "Rev.0.4"
- board text added: "VCC"
- board text removed: "Rev.0.3"

Commit message: before order pcbs
Parts:
- removed U4: TENDA_P200, openblw:TENDA_P200
- added JP4: M20-9990246, openblw:1X02
- added U$3: (no value), openblw:TENDA_P200
- C11: value 22u -> UUD1A220MCL1GS(22u)
- C15: value 10u -> UUD1E100MCL1GS(10u)
- F1: value MF-MSMF200 -> MF-MSMF200-2
- FB2, FB3: value FERRITE_BEAD -> 742792022
- IC6: value LAN9512 -> LAN9512-JZX
- JP1: value 90131-0764 -> M20-9980446
- JP2, JP3: value (none) -> M20-9980346; device pinhead:1X01 -> pinhead:2X03
- L1, L2: value 4.7u -> SRN4018-4R7M(4.7u)
- L3: value SRP1250A -> SRP1245A-100M
- U$2: value 282836-2 -> M20-9980346
- moved JP2 66.9 mm to (58.5, 10.4), turned to 90 degrees
- moved JP3 29.9 mm to (29.3, 29.5)
Connections:
- net +3V3: now also JP3.5, JP3.6, JP4.1; no longer JP2.1, U4.7, U4.8
- net AGND: now also JP2.5, JP2.6; no longer U4.5, U4.6
- net AVCC: now also JP2.1, JP2.2; no longer U4.1, U4.2
- net GND: now also JP4.2; no longer U4.12
Routing:
- net 3V3A1: track 66.8 -> 66.1 mm
- net GPIO47_1V8: track 39.6 -> 40.2 mm
- net EXT1/UART1_RX: track 48.1 -> 48.6 mm

Commit message: parts miss
Parts:
- FB1, FB4: value MI0805K601R-10 -> HR2220V801R-10
Changed lines of the file:
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@@
 </element>
 <element name="LOGO1" library="openblw" package="OHMYDIGIFAB_LOGO" value="" x="42.799" y="12.7"/>
-<element name="FB1" library="resistor" package="L5650M" value="MI0805K601R-10" x="68.072" y="19.304" smashed="yes" rot="R90">
+<element name="FB1" library="resistor" package="L5650M" value="HR2220V801R-10" x="68.072" y="19.304" smashed="yes" rot="R90">
 <attribute name="NAME" x="69.977" y="23.876" size="0.8128" layer="25" font="vector" rot="R90"/>
 </element>
@@
 <attribute name="VALUE" x="46.845" y="57.993" size="1.27" layer="27" rot="R180" display="off"/>
 </element>
-<element name="FB4" library="resistor" package="L5650M" value="MI0805K601R-10" x="61.976" y="19.304" smashed="yes" rot="R90">
+<element name="FB4" library="resistor" package="L5650M" value="HR2220V801R-10" x="61.976" y="19.304" smashed="yes" rot="R90">
 <attribute name="NAME" x="58.801" y="18.542" size="0.8128" layer="25" rot="R90"/>
 <attribute name="VALUE" x="66.421" y="17.399" size="1.27" layer="27" rot="R90" display="off"/>
