File: pcb/interface_board/interface_board.brd (EAGLE design)
At the start: 72 x 56 mm, 99 parts, among them IC1 V7805-1000, IC6 LAN9512-JZX, K1 61400416021, U1 SFW15R-1STE1LF, U2 SFW15R-1STE1LF, U3 DMG1012T, U5 PAM2306AYPKE

Commit message: ordered
Parts:
- moved C11 6.73 mm to (48.8, 31.4)
- moved C15 6.73 mm to (48.8, 26.3)
- moved IC1 6.35 mm to (40.3, 28.8)
Routing:
- net N$39: track 21.9 -> 15.5 mm
- net +5V: track 155.6 -> 152.1 mm
- net GND: track 54.1 -> 54.2 mm, vias 19 -> 219

Commit message: xo
Parts:
- removed R37: 12k, rcl:R0603
- added C44, C45: 20p, rcl:C0603
- added Q6: CTS_32X25_SMD, raspi:CTS_32X25
- added R19: 1M, rcl:R0603
- C4, C5: value NF -> 100p
- R2: value 0R -> 450K
- R3: value 0R -> 200K
- R4, R5: value NR -> 100K
- U5: value PAM2306AYPKE -> PAM2306DYPAA
- moved C42 5.54 mm to (25.1, 34.8), turned to 270 degrees
- moved C33 1.42 mm to (21.3, 35.7)
- moved R10 1.40 mm to (21.3, 33.7)
- moved C34 1.40 mm to (21.3, 37.7)
- moved C35 1.40 mm to (21.3, 39.8)
- moved C32 0.18 mm to (13.7, 26.9)
- moved C38 0.13 mm to (11.7, 26.9)
Connections:
- removed net GPIO6: IC6.12, R37.2
- new net LAN_RUN: IC6.12, PCB1.21
- net +3V3: now also PCB1.39, PCB1.40, PCB1.41, PCB1.42; no longer R37.1
- net +5V: no longer PCB1.39, PCB1.40, PCB1.41, PCB1.42
- net GND: now also C44.1, C45.1, PCB1.168
- net XI: now also C45.2, Q6.1, R19.2
- net XO: now also C44.2, Q6.3, R19.1
Routing:
- net LAN_RUN: track 0.00 -> 65.7 mm, vias 0 -> 3
- net +3V3: track 295.3 -> 339.2 mm, vias 17 -> 21
- net +5V: track 152.1 -> 117.6 mm, vias 7 -> 3
- net XI: track 0.00 -> 17.4 mm, vias 0 -> 1
- net XO: track 0.00 -> 11.0 mm, vias 0 -> 1
- net N$43: track 19.0 -> 27.8 mm
- net GPIO6: track 8.02 -> 0.00 mm, vias 1 -> 0
- net 3V3A1: track 66.1 -> 69.7 mm
- net RX_P: track 59.1 -> 60.4 mm
- net RX_N: track 56.0 -> 57.3 mm
- net TX_P: track 58.1 -> 59.0 mm
- net TX_N: track 63.4 -> 64.3 mm
- net GND: vias 219 -> 215
Other:
- board text added: "Rev.0.5"
- board text removed: "Rev.0.4"

Commit message: tune
Parts:
- moved LED2 1.40 mm to (5.84, 16.8)
- moved R15 1.40 mm to (2.92, 16.8)
- moved U3 1.27 mm to (5.61, 14.8)
- moved JP1 0.80 mm to (8.38, 10.3)
- moved PCB1 0.77 mm to (36.3, 18.8)
- moved U1 0.76 mm to (48.5, 8.26)
- moved U2 0.76 mm to (23.2, 8.26)
- moved JP2 0.68 mm to (58.8, 9.78)
- moved U$3 0.68 mm to (61.3, 5.97)
- moved JP3 0.68 mm to (29.6, 28.8)
- moved C14 0.65 mm to (13.5, 21.3)
- moved R7 0.63 mm to (5.08, 26.3)
- moved R8 0.63 mm to (7.11, 26.3)
- moved R9 0.63 mm to (9.14, 26.3)
- moved C13 0.52 mm to (13.5, 19.1)
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Routing:
- net GND: track 54.2 -> 65.5 mm, vias 215 -> 219
- net CM_VBAT: track 19.0 -> 20.8 mm
- net +3V3: track 339.2 -> 340.8 mm
- net CM_1V8: track 14.4 -> 15.5 mm
- net CAM1_IO1: track 46.4 -> 47.4 mm
- net EXT1/UART1_RX: track 48.6 -> 47.7 mm
- net CAM1_IO0: track 45.9 -> 46.9 mm
- net N$31: track 3.67 -> 4.59 mm
- net N$34: track 3.67 -> 4.57 mm
- net CM_3V3: track 18.1 -> 18.9 mm
- net LAN_RUN: track 65.7 -> 66.5 mm
- net CAM1_SDA: track 52.3 -> 53.1 mm
- net CAM0_SDA: track 22.8 -> 22.1 mm
- net USB_D_N: track 19.8 -> 20.6 mm
- net CAM0_SCL: track 23.1 -> 22.4 mm
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Other:
- board text added: "*"

Commit message: interface_board
Parts:
- added JP5: USB-IDMICRO, openblw:USB-MICRO
Connections:
- new net N$47: IC6.1, JP5.D-
- new net N$48: IC6.2, JP5.D+
- net +5V: now also JP5.VBUS
- net GND: now also JP5.GND
