File: pcb/interface_board/interface_board.sch (EAGLE design)
At the start: 57 parts, among them CN1 B2B-PH-K-S, IC1 V7805-1000, K1 61400416021, U1 SFW15R-1STE1LF, U2 SFW15R-1STE1LF, U3 DMG1012T, U4 TENDA_P200, U5 PAM2306AYPKE, U6 AP7115-25SEG

Commit message: client board
Parts:
- removed C10: 4.7u, resistor:C-EUC0603
- removed C8: 1u, resistor:C-EUC0402
- removed C9: 100n, resistor:C-EUC0402
- removed CN1: B2B-PH-K-S, openblw:JST_2PIN-THM
- removed R10: 0R, resistor:R-EU_R0805
- removed U6: AP7115-25SEG, openblw:AP7115-XXSEG
- added U$1, U$2: 282836-2, openblw:282836-2
- FB1: device openblw:FERRITESIZE_0805 -> resistor:L-EUL5650M
- L3: device openblw:BOURNS-SRN4018 -> openblw:SRP1250
Connections:
- removed net +2V5: C10.1, R10.2, U6.OUT@5
- removed net CM_VDAC: PCB1.189/VDAC, PCB1.190/VDAC, R10.1
- removed net N$37: C16.1, F1.1, L3.1
- removed net N$5: C9.1, U6.BP@4
- new net N$39: C15.+, F1.2, IC1.IN
- net +12V: now also C16.1, F1.1, L3.1, U$2.CON01; no longer C15.+, F1.2, IC1.IN
- net +3V3: no longer C8.1, PCB1.39/GPIO0-27_VREF, PCB1.40/GPIO0-27_VREF, PCB1.41/GPIO28-45_VREF, PCB1.42/GPIO28-45_VREF, U6.EN@3, U6.IN@1
- net +5V: now also PCB1.39/GPIO0-27_VREF, PCB1.40/GPIO0-27_VREF, PCB1.41/GPIO28-45_VREF, PCB1.42/GPIO28-45_VREF
- net CM_3V3: now also PCB1.189/VDAC, PCB1.190/VDAC
- net GND: now also U$1.CON02, U$2.CON02; no longer C10.2, C8.2, C9.2, CN1.1, U6.GND@2
- net N$36: now also U$1.CON01; no longer CN1.2
Other:
- moved on the sheet: C16

Commit message: rj45
Parts:
- added ETH1: HR911105A, openblw:HR911105A
- L3: value 10u -> SRP1250A; device openblw:SRP1250 -> openblw:SRP1250A
Connections:
- net +12V: now also L3.2; no longer L3.1
- net N$6: now also L3.1; no longer L3.2
Changed lines of the file:
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@@
 <part name="C15" library="resistor" deviceset="CPOL-EU" device="153CLV-0405" value="10u"/>
 <part name="FB1" library="resistor" deviceset="L-EU" device="L5650M" value="MI0805K601R-10"/>
-<part name="L3" library="openblw" deviceset="SRP1250" device="" value="10u"/>
 <part name="C16" library="resistor" deviceset="C-EU" device="C0402" value="1u"/>
 <part name="R18" library="resistor" deviceset="R-EU_" device="R0402" value="1K"/>
@@
 <part name="V33" library="supply" deviceset="+12V" device=""/>
 <part name="GND31" library="supply" deviceset="GND" device=""/>
+<part name="ETH1" library="openblw" deviceset="HR911105A" device=""/>
+<part name="L3" library="openblw" deviceset="SRP1250A" device=""/>
 </parts>
 <sheets>
@@
 <instance part="C15" gate="G$1" x="109.22" y="208.28"/>
 <instance part="FB1" gate="G$1" x="33.02" y="213.36" rot="R90"/>
-<instance part="L3" gate="G$1" x="55.88" y="213.36" rot="MR0"/>
 <instance part="C16" gate="G$1" x="68.58" y="208.28"/>
 <instance part="R18" gate="G$1" x="43.18" y="205.74" rot="R270"/>
@@
 <instance part="V33" gate="1" x="233.68" y="165.1"/>
 <instance part="GND31" gate="1" x="238.76" y="165.1" rot="R180"/>
+<instance part="ETH1" gate="G$1" x="195.58" y="66.04"/>
+<instance part="L3" gate="G$1" x="55.88" y="213.36"/>
 </instances>
 <busses>
@@
 <segment>
 <pinref part="FB1" gate="G$1" pin="2"/>
-<pinref part="L3" gate="G$1" pin="2"/>
 <wire x1="38.1" y1="213.36" x2="43.18" y2="213.36" width="0.1524" layer="91"/>
 <pinref part="R18" gate="G$1" pin="1"/>
@@
 <wire x1="43.18" y1="210.82" x2="43.18" y2="213.36" width="0.1524" layer="91"/>
 <junction x="43.18" y="213.36"/>
+<pinref part="L3" gate="G$1" pin="1"/>
 </segment>
 </net>
@@
 <net name="+12V" class="5">
 <segment>
-<pinref part="L3" gate="G$1" pin="1"/>
 <pinref part="F1" gate="G$1" pin="1"/>
 <wire x1="60.96" y1="213.36" x2="68.58" y2="213.36" width="0.1524" layer="91"/>
@@
 <wire x1="76.2" y1="220.98" x2="76.2" y2="213.36" width="0.1524" layer="91"/>
 <junction x="76.2" y="213.36"/>
-</segment>
-<segment>
+<pinref part="L3" gate="G$1" pin="2"/>
+</segment>
+<segment>

Commit message: lan
Parts:
- removed ETH1: HR911105A, openblw:HR911105A
- added C10, C41: 10u, rcl:C-EUC0805
- added C21, C22, C23, C24: 20p, rcl:C-EUC0603
- added C26, C27, C28, C29, C30, C31, C32, C33, C34, C35, C36, C37, C38, C39, C40, C43, C8, C9: 100n, rcl:C-EUC0603
- added C42: 1u, rcl:C-EUC0805
- added ETHERNET: HR911105A, hanrun:HR911105A
- added FB2, FB3: FERRITE_BEAD, raspi:FERRITE_BEAD
- added FB4: MI0805K601R-10, resistor:L-EUL5650M
- added IC6: LAN9512, raspi:LAN9512
- added JP2, JP3: (no value), pinhead:PINHD-1X1
- added R10, R20, R32, R37: 12k, rcl:R-EU_R0603
- added R25, R26: 1k, rcl:R-EU_R0603
- added R27: 10, rcl:R-EU_R0603
- added R28, R29, R30, R31: 49.9, rcl:R-EU_R0603
- added R33: 12k4, rcl:R-EU_R0603
Connections:
- removed net N$36: FB1.1, U$1.CON01
- removed net PLC_N: U4.INN
- removed net PLC_P: U4.INP
- new net 3V3A: C8.1, C9.1, R27.1, R28.1, R29.1, R30.1, R31.1
- new net 3V3A1: C32.2, C33.2, C34.2, C35.2, C36.2, C37.2, C38.2, FB2.P$1, IC6.VDD33A@1, IC6.VDD33A@2, IC6.VDD33A@3, IC6.VDD33A@4, IC6.VDD33A@5, IC6.VDD33A@6, IC6.VDD33A@7
- new net AGND: FB4.1, U$1.CON01, U4.INN
- new net AVCC: FB1.1, U$1.CON02, U4.INP
- new net GPIO6: IC6.NRESET, R37.2
- new net N$37: ETHERNET.P$12, R25.2
- new net N$40: ETHERNET.P$9, R26.2
- new net N$41: C26.1, ETHERNET.P$4, ETHERNET.P$5, R27.2
- new net N$42: IC6.USBRBIAS, R10.2
- new net N$43: C42.2, FB3.P$2, IC6.VDD18USBPLL
- new net N$44: IC6.AUTOMDXI_EN, R32.1
- new net N$45: IC6.EXRES, R33.1
- new net N$46: IC6.NTRST, R20.1
- new net NLNKA_LED: ETHERNET.P$10, IC6.NLNKA_LED/GPIO1
- new net NSPD_LED: ETHERNET.P$11, IC6.NSPD_LED/GPIO2
- new net RX_N: C24.1, ETHERNET.P$6, IC6.RXN, R28.2
- new net RX_P: C23.1, ETHERNET.P$3, IC6.RXP, R29.2
- new net TX_N: C22.1, ETHERNET.P$2, IC6.TXN, R30.2
- new net TX_P: C21.1, ETHERNET.P$1, IC6.TXP, R31.2
- new net USBD3_N: IC6.USBDM3, K1.D-
- new net USBD3_P: IC6.USBDP3, K1.D+
- new net VDD18CORE: C39.2, C40.2, C41.2, IC6.VDD18CORE@1, IC6.VDD18CORE@2
- new net VDD18PLL: C43.2, FB3.P$1, IC6.VDD18ETHPLL
- new net XI: IC6.XI
- new net XO: IC6.XO
- net +3V3: now also C27.1, C28.1, C29.1, C30.2, C31.2, FB2.P$2, IC6.TEST3, IC6.VBUS_DET, IC6.VDD33IO@1, IC6.VDD33IO@2, IC6.VDD33IO@3, IC6.VDD33IO@4, IC6.VDD33IO@5, JP2.1, R20.2, R25.1, R26.1, R32.2, R37.1
- net +5V: now also C10.1
- net GND: now also C10.2, C21.2, C22.2, C23.2, C24.2, C26.2, C27.2, C28.2, C29.2, C30.1, C31.1, C32.1, C33.1, C34.1, C35.1, C36.1, C37.1, C38.1, C39.1, C40.1, C41.1, C42.1, C43.1, C8.2, C9.2, ETHERNET.P$8, FB4.2, IC6.CLK24_EN, IC6.GND, IC6.TEST2, JP3.1, R10.1, R33.2; no longer U$1.CON02
- net USB_D_N: now also IC6.USBDM0; no longer K1.D-
- net USB_D_P: now also IC6.USBDP0; no longer K1.D+

Commit message: before order pcbs
Parts:
- removed U4: TENDA_P200, openblw:TENDA_P200
- added JP4: M20-9990246, openblw:PINHD-1X2
- C11: value 22u -> UUD1A220MCL1GS(22u)
- C15: value 10u -> UUD1E100MCL1GS(10u)
- F1: value MF-MSMF200 -> MF-MSMF200-2
- FB2, FB3: value FERRITE_BEAD -> 742792022
- IC6: value LAN9512 -> LAN9512-JZX
- JP1: value 90131-0764 -> M20-9980446
- JP2, JP3: value (none) -> M20-9980346; device pinhead:PINHD-1X1 -> pinhead:PINHD-2X3
- L1, L2: value 4.7u -> SRN4018-4R7M(4.7u)
- L3: value SRP1250A -> SRP1245A-100M
- U$2: value 282836-2 -> M20-9980346
Connections:
- net +3V3: now also JP3.5, JP3.6, JP4.1; no longer JP2.1, U4.3V3
- net AGND: now also JP2.5, JP2.6; no longer U4.INN
- net AVCC: now also JP2.1, JP2.2; no longer U4.INP
- net GND: now also JP4.2; no longer U4.GND
Other:
- moved on the sheet: C10, C21, C22, C23, C24, C26, C27, C28, C29, C30, C31, C32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

Commit message: parts miss
Parts:
- FB1, FB4: value MI0805K601R-10 -> HR2220V801R-10
Changed lines of the file:
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@@
 <part name="FRAME1" library="frames" deviceset="A3L-LOC" device=""/>
 <part name="C15" library="resistor" deviceset="CPOL-EU" device="153CLV-0405" value="UUD1E100MCL1GS(10u)"/>
-<part name="FB1" library="resistor" deviceset="L-EU" device="L5650M" value="MI0805K601R-10"/>
+<part name="FB1" library="resistor" deviceset="L-EU" device="L5650M" value="HR2220V801R-10"/>
 <part name="C16" library="resistor" deviceset="C-EU" device="C0402" value="1u"/>
 <part name="R18" library="resistor" deviceset="R-EU_" device="R0402" value="1K"/>
@@
 <part name="R37" library="rcl" deviceset="R-EU_" device="R0603" value="12k"/>
 <part name="K1" library="openblw" deviceset="61400416021" device=""/>
-<part name="FB4" library="resistor" deviceset="L-EU" device="L5650M" value="MI0805K601R-10"/>
+<part name="FB4" library="resistor" deviceset="L-EU" device="L5650M" value="HR2220V801R-10"/>
 <part name="V6" library="supply" deviceset="+3V3" device=""/>
 <part name="GND10" library="supply" deviceset="GND" device=""/>

Commit message: xo
Parts:
- removed R37: 12k, rcl:R-EU_R0603
- added C44, C45: 20p, rcl:C-EUC0603
- added Q6: CTS_32X25_SMD, raspi:CTS_32X25_SMD
- added R19: 1M, rcl:R-EU_R0603
- C4, C5: value NF -> 100p
- R2: value 0R -> 450K
- R3: value 0R -> 200K
- R4, R5: value NR -> 100K
- U5: value PAM2306AYPKE -> PAM2306DYPAA
Connections:
- removed net GPIO6: IC6.NRESET, R37.2
- new net LAN_RUN: IC6.NRESET, PCB1.21/GPIO6
- net +3V3: now also PCB1.39/GPIO0-27_VREF, PCB1.40/GPIO0-27_VREF, PCB1.41/GPIO28-45_VREF, PCB1.42/GPIO28-45_VREF; no longer R37.1
- net +5V: no longer PCB1.39/GPIO0-27_VREF, PCB1.40/GPIO0-27_VREF, PCB1.41/GPIO28-45_VREF, PCB1.42/GPIO28-45_VREF
- net GND: now also C44.1, C45.1, PCB1.168/USB_OTGID
- net XI: now also C45.2, Q6.X1, R19.2
- net XO: now also C44.2, Q6.X2, R19.1
Other:
- moved on the sheet: R11, R12

Commit message: interface_board
Parts:
- added JP5: USB-IDMICRO, openblw:USB-IDMICRO
Connections:
- new net N$47: IC6.USBDM2, JP5.D-
- new net N$48: IC6.USBDP2, JP5.D+
- net +5V: now also JP5.VBUS
- net GND: now also JP5.GND
Changed lines of the file:
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@@
 <part name="Q6" library="raspi" deviceset="CTS_32X25_SMD" device=""/>
 <part name="GND53" library="supply1" deviceset="GND" device=""/>
+<part name="JP5" library="openblw" deviceset="USB-ID" device="MICRO"/>
 </parts>
 <sheets>
@@
 <instance part="C10" gate="G$1" x="294.64" y="60.96"/>
 <instance part="GND9" gate="1" x="294.64" y="50.8"/>
-<instance part="GND12" gate="1" x="276.86" y="66.04" rot="R180"/>
+<instance part="GND12" gate="1" x="210.82" y="60.96"/>
 <instance part="P+8" gate="1" x="299.72" y="66.04" rot="R270"/>
 <instance part="GND32" gate="1" x="317.5" y="91.44"/>
@@
 <instance part="Q6" gate="G$2" x="175.26" y="68.58" rot="R90"/>
 <instance part="GND53" gate="1" x="157.48" y="73.66" rot="R270"/>
+<instance part="JP5" gate="G$1" x="241.3" y="55.88" rot="R270"/>
 </instances>
 <busses>
@@
 <pinref part="GND12" gate="1" pin="GND"/>
 <pinref part="K1" gate="G$1" pin="GND"/>
+<wire x1="210.82" y1="63.5" x2="241.3" y2="63.5" width="0.1524" layer="91"/>
+<pinref part="JP5" gate="G$1" pin="GND"/>
+<wire x1="241.3" y1="63.5" x2="276.86" y2="63.5" width="0.1524" layer="91"/>
+<wire x1="241.3" y1="58.42" x2="241.3" y2="63.5" width="0.1524" layer="91"/>
+<junction x="241.3" y="63.5"/>
 </segment>
 <segment>
@@
 <junction x="294.64" y="66.04"/>
 <pinref part="K1" gate="G$1" pin="VCC"/>
+<pinref part="JP5" gate="G$1" pin="VBUS"/>
+<wire x1="243.84" y1="58.42" x2="243.84" y2="66.04" width="0.1524" layer="91"/>
+<wire x1="243.84" y1="66.04" x2="284.48" y2="66.04" width="0.1524" layer="91"/>
+<junction x="284.48" y="66.04"/>
 </segment>
 </net>
@@
 </segment>
 </net>
+<net name="N$47" class="0">
+<segment>
+<pinref part="JP5" gate="G$1" pin="D-"/>
+<wire x1="246.38" y1="58.42" x2="246.38" y2="78.74" width="0.1524" layer="91"/>
+<pinref part="IC6" gate="G$1" pin="USBDM2"/>
+<wire x1="246.38" y1="78.74" x2="256.54" y2="78.74" width="0.1524" layer="91"/>
+<wire x1="256.54" y1="78.74" x2="256.54" y2="86.36" width="0.1524" layer="91"/>
+</segment>
+</net>
+<net name="N$48" class="0">
+<segment>
+<pinref part="JP5" gate="G$1" pin="D+"/>
+<wire x1="248.92" y1="58.42" x2="248.92" y2="76.2" width="0.1524" layer="91"/>
+<pinref part="IC6" gate="G$1" pin="USBDP2"/>
+<wire x1="248.92" y1="76.2" x2="259.08" y2="76.2" width="0.1524" layer="91"/>
+<wire x1="259.08" y1="76.2" x2="259.08" y2="86.36" width="0.1524" layer="91"/>
+</segment>
+</net>
